File: とある自作の回路群/Railgun_Boost-circuit/Railgun_Boost-circuit.kicad_pcb (KiCad board)
At the start: 2 copper layers, 73 parts, among them IC1 CH221K, IC2 TLP152, J1 USB_C_Receptacle_USB2.0, J2 XH2P, J3 XH2P, J4 XH2P, J5 XH4P, K1 DG85B-7011-75-1012, Q1 FDS4935A, Q2 FDS4935A, Q3 NMOS, Q4 FDS4935A, Q5 NMOS, Q6 NMOS, U1 L7805, U2 74HC21, U3 NJM2903, U4 NJM4558, U5 NJM2903

Commit message: PCB入り
Parts:
- removed Q5: NMOS, samasys:TK042N65Z5
- removed Q6: NMOS, Package_TO_SOT_SMD:TSOT-23
- added HS1: Heatsink_Pad_2Pin, Mylibrary:20PB020-01025, F.Cu at (170.3, 73.5)
- added HS2: Heatsink_Pad_2Pin, Mylibrary:20PB020-01025, F.Cu at (166.3, 91.7)
- F1: footprint samasys:3557-2 -> Fuse:Fuse_Bourns_MF-RG300
- Q1, Q4: value FDS4935A -> NMOS; footprint samasys:SOIC127P600X175-8N -> Package_TO_SOT_SMD:TSOT-23
- Q2: value FDS4935A -> PMOS; footprint samasys:SOIC127P600X175-8N -> Package_TO_SOT_SMD:TO-252-2
- Q3: footprint Package_TO_SOT_SMD:TSOT-23 -> samasys:TK042N65Z5
- R10: value 1.5k -> 4.7k
- R11: value 4.7k -> 510; footprint Resistor_SMD:R_0603_1608Metric -> Resistor_THT:R_Axial_DIN0204_L3.6mm_D1.6mm_P5.08mm_Horizontal
- R12: value 510 -> 10k; footprint Resistor_THT:R_Axial_DIN0204_L3.6mm_D1.6mm_P5.08mm_Horizontal -> Resistor_SMD:R_0603_1608Metric
- R13: value 10k -> 1k
- R14: value 1k -> 20k; footprint Resistor_SMD:R_0603_1608Metric -> Resistor_THT:R_Axial_DIN0204_L3.6mm_D1.6mm_P5.08mm_Horizontal
- R15: value 20k -> 1.5k
- R16: value 1.6k -> 10k; footprint Resistor_THT:R_Axial_DIN0204_L3.6mm_D1.6mm_P5.08mm_Horizontal -> Resistor_SMD:R_0603_1608Metric
- R27, R28: footprint Resistor_SMD:R_0603_1608Metric -> Resistor_THT:R_Axial_DIN0207_L6.3mm_D2.5mm_P10.16mm_Horizontal
- R9: value 10k -> 1.5k
- moved K1 143.2 mm to (241.2, 80.7)
- moved IC1 130.3 mm to (11.8, 110.0)
- moved R14 122.4 mm to (2.60, 89.1)
- moved R11 117.1 mm to (2.60, 86.0)
- moved Q3 91.2 mm to (164.9, 79.8)
- moved Q1 89.5 mm to (43.0, 94.6)
- moved RV1 89.4 mm to (52.2, 51.0)
- moved RV2 89.4 mm to (58.1, 51.0)
- moved RV3 89.4 mm to (64.0, 51.0)
- moved Q4 87.8 mm to (43.0, 99.2)
- moved U2 79.7 mm to (38.0, 74.8)
- moved R18 79.2 mm to (52.2, 59.6)
- moved U1 77.8 mm to (54.6, 110.3)
- moved R15 75.2 mm to (2.60, 92.2)
- moved J2 75.1 mm to (12.6, 87.8)
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Connections:
- F1 pad 1: +BATT -> VBUS
- IC2 pad 3: Net-(Q3-D) -> Net-(Q1-D)
- J1 pad A4: +12V -> VBUS
- J1 pad A9: +12V -> VBUS
- J1 pad B4: +12V -> VBUS
- J1 pad B9: +12V -> VBUS
- J2 pad 1: /PowerSIG -> +5V
- J2 pad 2: GND -> /ChargeSIG
- J3 pad 1: +5V -> /PowerSIG
- J3 pad 2: /ChargeSIG -> GND
- L1 pad 1: Net-(L1-Pad1) -> Net-(Q2-D)
- Q1 pad 1: +24V -> Net-(Q1-D)
- Q1 pad 2: /PowerSIG -> Net-(Q1-G)
- Q1 pad 3: +24V -> GND
- Q2 pad 1: +24V -> Net-(Q2-D)
- Q3 pad 1: Net-(Q3-D) -> Net-(D6-A)
- Q3 pad 3: GND -> /CapV-_Sence
- Q4 pad 1: +24V -> Net-(D7-A)
- Q4 pad 2: /PowerSIG -> Net-(Q4-G)
- Q4 pad 3: +24V -> GND
- R10 pad 2: /PFM -> /OCP
- R11 pad 1: +5V -> /OCP
- R11 pad 2: /OCP -> Net-(U3B-+)
- R12 pad 1: /OCP -> Net-(Q1-G)
- R12 pad 2: Net-(U3B-+) -> GND
- R13 pad 1: Net-(Q3-G) -> +12V
- R13 pad 2: GND -> Net-(IC2-Pad1)
- R14 pad 2: Net-(IC2-Pad1) -> /PFM
- R15 pad 2: /PFM -> Net-(U3B-+)
- R16 pad 1: +12V -> +24V
- R16 pad 2: Net-(U3B-+) -> /PowerSIG
- R18 pad 2: Net-(Q5-G) -> Net-(Q3-G)
- R20 pad 1: Net-(Q5-G) -> Net-(Q3-G)
- R3 pad 1: +12V -> VBUS
- R30 pad 1: Net-(Q6-G) -> Net-(Q4-G)
- R9 pad 1: +24V -> +5V
- R9 pad 2: /PowerSIG -> /PFM
- U2 pad 6: Net-(Q3-G) -> Net-(Q1-G)
- U2 pad 8: Net-(Q6-G) -> Net-(Q4-G)
Other:
- board outline added: 100 x 50 mm

Commit message: 回路図完成、Desktopに引き継ぎ
Parts:
- removed R35: 1M, Resistor_SMD:R_0805_2012Metric
- added D10: LED, LED_SMD:LED_0603_1608Metric, F.Cu at (173.6, 48.8)
- added D11: LED, LED_SMD:LED_0603_1608Metric, F.Cu at (181.8, 41.7)
- added D8: LED, LED_SMD:LED_0603_1608Metric, F.Cu at (173.6, 43.6)
- added D9: LED, LED_SMD:LED_0603_1608Metric, F.Cu at (173.6, 46.2)
- added R36: 1.5k, Resistor_SMD:R_0603_1608Metric, F.Cu at (181.8, 46.8)
- added R37: 5.1k, Resistor_SMD:R_0603_1608Metric, F.Cu at (188.2, 45.6)
- added REF**: MountingHole_3.2mm_M3, MountingHole:MountingHole_3.2mm_M3, F.Cu at (196.6, 53.5)
- added REF**: MountingHole_3.2mm_M3, MountingHole:MountingHole_3.2mm_M3, F.Cu at (103.5, 53.5)
- added REF**: MountingHole_3.2mm_M3, MountingHole:MountingHole_3.2mm_M3, F.Cu at (103.5, 101.0)
- added REF**: MountingHole_3.2mm_M3, MountingHole:MountingHole_3.2mm_M3, F.Cu at (196.6, 101.0)
- D1, D2: footprint samasys:MA10EB045 -> samacsys:CUHS20F30H3F
- D6: footprint Mylibrary:PCDP0665G1 -> MyLibrary:PCDP0665G1
- D7: footprint samasys:MA10EB045 -> samacsys:CUHS20F30H3F; moved to B.Cu
- F1: footprint Fuse:Fuse_Bourns_MF-RG300 -> Fuse:Fuse_Bourns_MF-RG1000
- F2: footprint samasys:3557-2 -> samacsys:3557-2
- HS1: value Heatsink_Pad_2Pin -> For Q3; footprint Mylibrary:20PB020-01025 -> MyLibrary:20PB020-01025
- HS2: value Heatsink_Pad_2Pin -> For D6; footprint Mylibrary:20PB020-01025 -> MyLibrary:20PB020-01025
- IC1: footprint samasys:SOT95P280X120-6N -> samacsys:SOT95P280X120-6N
- IC2: footprint samasys:11-4L1S_5-PIN-SOIC_ -> samacsys:11-4L1S_5-PIN-SOIC_
- J5: value XH4P -> XT30PW-F; footprint Connector_JST:JST_XH_B4B-XH-A_1x04_P2.50mm_Vertical -> Connector_AMASS:AMASS_XT30PW-F_1x02_P2.50mm_Horizontal
- K1: value DG85B-7011-75-1012 -> G6B-1114P-US-DC12; footprint samasys:DG85B7011751024 -> samacsys:G6B1114PUSDC12
- L1: value L -> 90u; footprint samasys:HK12S1009000 -> samacsys:HK12S1009000
- Q1: value NMOS -> Q_NMOS
- Q2: value PMOS -> Q_PMOS
- Q3: value NMOS -> Q_NMOS; footprint samasys:TK042N65Z5 -> samacsys:TK042N65Z5
- Q4: value NMOS -> Q_NMOS; moved to B.Cu
- R1, R2, R20, R25, R30, R32, R4, R5, R7: moved to B.Cu
- R11, R17, R19, R33: footprint Resistor_THT:R_Axial_DIN0204_L3.6mm_D1.6mm_P5.08mm_Horizontal -> Resistor_SMD:R_0603_1608Metric; moved to B.Cu
- R14, R15, R21, R22, R26, R29: footprint Resistor_THT:R_Axial_DIN0204_L3.6mm_D1.6mm_P5.08mm_Horizontal -> Resistor_SMD:R_0603_1608Metric
- R16: value 10k -> 5.1k
- R18: footprint Resistor_THT:R_Axial_DIN0207_L6.3mm_D2.5mm_P10.16mm_Horizontal -> Resistor_SMD:R_0603_1608Metric; moved to B.Cu
- R23: footprint samasys:RESM6331X120N -> samacsys:RESM6331X120N; moved to B.Cu
- R27, R28: value 150k -> 100k; footprint Resistor_THT:R_Axial_DIN0207_L6.3mm_D2.5mm_P10.16mm_Horizontal -> Resistor_SMD:R_0603_1608Metric; moved to B.Cu
- R31: value 1M -> 1.5; footprint Resistor_SMD:R_0805_2012Metric -> Resistor_SMD:R_0603_1608Metric
- R34: value 1M -> 1.5k; footprint Resistor_SMD:R_0805_2012Metric -> Resistor_SMD:R_0603_1608Metric
- moved R33 199.2 mm to (195.0, 62.7), turned to 90 degrees
- moved R26 194.5 mm to (194.0, 73.2), turned to 180 degrees
- moved R29 192.1 mm to (190.9, 73.2)
- moved J5 175.1 mm to (191.8, 61.7), turned to -90 degrees
- moved U5 171.3 mm to (197.6, 75.6), turned to -90 degrees
- moved R32 159.8 mm to (195.0, 66.0), turned to 90 degrees
- moved D5 152.8 mm to (185.0, 53.4), turned to 90 degrees
- moved R34 149.3 mm to (177.6, 46.1)
- moved R31 148.1 mm to (177.6, 43.6)
- moved D3 144.8 mm to (178.4, 53.4), turned to -90 degrees
- moved R22 142.4 mm to (142.8, 79.8)
- moved R21 142.3 mm to (142.8, 77.0)
- moved R24 141.1 mm to (198.4, 73.2), turned to 180 degrees
- moved R14 139.8 mm to (142.4, 87.2), turned to -90 degrees
- moved U3 138.0 mm to (139.8, 93.2), turned to 180 degrees
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Connections:
- IC1 pad 3: unconnected-(IC1-PG-Pad3) -> /PG
- J3 pad 2: GND -> Net-(J3-Pin_2)
- J5 pad 1: /CapV+_Sence -> /CapV-_Sence
- Q1 pad 1: Net-(Q1-D) -> Net-(Q1-G)
- Q1 pad 2: Net-(Q1-G) -> GND
- Q1 pad 3: GND -> Net-(Q1-D)
- Q2 pad 1: Net-(Q2-D) -> /PowerSIG
- Q2 pad 2: /PowerSIG -> Net-(Q2-D)
- Q3 pad 1: Net-(D6-A) -> Net-(Q3-G)
- Q3 pad 2: Net-(Q3-G) -> Net-(D6-A)
- Q4 pad 1: Net-(D7-A) -> Net-(Q4-G)
- Q4 pad 2: Net-(Q4-G) -> GND
- Q4 pad 3: GND -> Net-(D7-A)
- R31 pad 1: /CapV+_Sence -> Net-(D9-K)
- R31 pad 2: Net-(R31-Pad2) -> GND
- R32 pad 1: Net-(R31-Pad2) -> /CapV+_Sence
- R34 pad 1: /CapV+_Sence -> Net-(D10-K)
- R34 pad 2: Net-(R34-Pad2) -> GND
- U3 pad 4: +12V -> GND
- U3 pad 8: GND -> +12V
- U5 pad 4: +12V -> GND
- U5 pad 8: GND -> +12V
Routing:
- net Net-(D5-K): vias 0 -> 1
- net Net-(D4-K): vias 0 -> 1
- net Net-(D3-K): vias 0 -> 1
Other:
- board size 100 x 50 mm -> 100 x 54.6 mm
